File: hardwired/oscilator/clean_pwm_saw/clean_pwm_saw.kicad_sch (KiCad schematic)
At the start: 0 parts

Commit message: Massive dump of circuits and code
Parts:
- added C1: 10n, symbol Device:C
- added D1, D2, D3, D4: D, symbol Device:D
- added Q1, Q4: NPN, symbol Simulation_SPICE:NPN
- added Q2, Q3: PNP, symbol Simulation_SPICE:PNP
- added R1: Potentiometer, symbol Simulation_SPICE:Potentiometer
- added R2, R5: 47k, symbol Device:R
- added R3, R4: 33k, symbol Device:R
- added R6: 18k, symbol Device:R
- added R7: 10k, symbol Device:R
- added R8: 47, symbol Device:R
- added U1, U2, U3: ${SIM.PARAMS}, symbol Simulation_SPICE:OPAMP
- added V1, V2: 12, symbol Simulation_SPICE:VDC
Connections:
- new net: D1.2 (A), D3.2 (A), Q3.1 (C)
- new net: Q1.1 (C), Q2.1 (C), Q2.2 (B), Q3.2 (B)
- new net: R2.1, R6.1, U2.1 (+)
- new net: Q4.3 (E), R7.1, U2.2 (-)
- new net: Q1.2 (B), U1.5
- new net: Q1.3 (E), R5.1, U1.2 (-)
- new net: C1.1, R8.2
- new net +12V: Q2.3 (E), Q3.3 (E), R1.1, U1.3 (V+), U2.3 (V+), U3.3 (V+), V1.1
- new net -12V: R6.2, R7.2, U1.4 (V-), U2.4 (V-), U3.4 (V-), V2.2
- new net 0: C1.2, R1.3, R2.2, R3.2, R5.2, V1.2, V2.1
- new net CAP: D1.1 (K), D4.2 (A), R8.1, U3.2 (-)
- new net CV: R1.2, U1.1 (+)
- new net SINK: D2.1 (K), D4.1 (K), Q4.1 (C)
- new net SQ: D2.2 (A), D3.1 (K), R4.2, U3.5
- new net THRESH: R3.1, R4.1, U3.1 (+)
- new net U2_OUT: Q4.2 (B), U2.5
