File: hardwired/oscilator/saw_triangle_morph/saw_triangle_morph.kicad_sch (KiCad schematic)
At the start: 21 parts, among them Q1 PNP, Q2 NPN, U1 ${SIM.PARAMS}, U2 ${SIM.PARAMS}

Commit message: Massive dump of circuits and code
Parts:
- removed C2, C3: 1000u, Connector_PinSocket_2.54mm:PinSocket_1x02_P2.54mm_Vertical, symbol Device:C_Polarized
- removed Q2: NPN, Connector_PinSocket_2.54mm:PinSocket_1x03_P2.54mm_Vertical, symbol Simulation_SPICE:NPN
- removed R10: 56k, Resistor_THT:R_Axial_DIN0411_L9.9mm_D3.6mm_P15.24mm_Horizontal, symbol Device:R
- removed R11, R12: 10k, Resistor_THT:R_Axial_DIN0411_L9.9mm_D3.6mm_P15.24mm_Horizontal, symbol Device:R
- removed R4: 3.3k, Resistor_THT:R_Axial_DIN0309_L9.0mm_D3.2mm_P15.24mm_Horizontal, symbol Device:R
- removed R8: Potentiometer, Connector_PinHeader_2.54mm:PinHeader_1x03_P2.54mm_Horizontal, symbol Simulation_SPICE:Potentiometer
- added D3, D4: D, symbol Device:D
- added Q2: BC327, symbol Simulation_SPICE:PNP
- added Q4, Q5: BC337, symbol Simulation_SPICE:NPN
- added R4: Potentiometer, symbol Simulation_SPICE:Potentiometer
- added R7: 33k, symbol Device:R
- added R8: 47, symbol Device:R
- added U3: ${SIM.PARAMS}, symbol Simulation_SPICE:OPAMP
- C1: value 0.01u -> 1n
- D1, D2: footprint Diode_THT:D_A-405_P7.62mm_Horizontal -> (none)
- Q1: value PNP -> BC327; footprint Connector_PinSocket_2.54mm:PinSocket_1x03_P2.54mm_Vertical -> (none)
- R1: value 8.2 -> 12k; footprint Resistor_THT:R_Axial_DIN0309_L9.0mm_D3.2mm_P15.24mm_Horizontal -> (none)
- R2: value 8.2 -> 47k; footprint Resistor_THT:R_Axial_DIN0309_L9.0mm_D3.2mm_P15.24mm_Horizontal -> (none)
- R3: value 3.3k -> 10k; footprint Resistor_THT:R_Axial_DIN0309_L9.0mm_D3.2mm_P15.24mm_Horizontal -> (none)
- R5: footprint Resistor_THT:R_Axial_DIN0309_L9.0mm_D3.2mm_P15.24mm_Horizontal -> (none)
- R6: value 33k -> 470k; footprint Resistor_THT:R_Axial_DIN0309_L9.0mm_D3.2mm_P15.24mm_Horizontal -> (none)
- U1, U2: footprint Package_DIP:DIP-8_W7.62mm -> (none)
Connections:
- net +12V: now also Q1.3 (E), Q2.3 (E), R4.3, U3.3 (V+); no longer R3.1, R5.1
- net -12V: now also R1.2, R3.2, U3.4 (V-); no longer Q1.1 (C), R6.2
- net 0: now also C1.2, R2.1, R6.2, R4.1, R7.1
- net SQ: now also R5.2, D3.2 (A), D4.1 (K), U3.5; no longer U2.5
- net at U1.1 (+): now also R4.2
- net CAP: now reaches D1.1 (K), D2.2 (A)
- net CAP: now also R8.1, U3.2 (-); no longer U1.5
- net I_CHARGE: now reaches D1.2 (A)
- net I_CHARGE: now also Q1.1 (C), D4.2 (A); no longer R3.2
- net at R1.1: now also U2.2 (-), Q4.3 (E)
- net at U2.1 (+): now also R2.2, R3.1
- net at Q1.2 (B): now also Q2.1 (C), Q2.2 (B), Q5.1 (C); no longer D2.1 (K)
- net at R6.1: now also U1.2 (-), Q5.3 (E)
- removed net TRI: C1.2, U2.2 (-)
- removed net VGND: C1.1, R1.2, R2.1, U1.2 (-)
- new net: C1.1, R8.2
- new net: Q5.2 (B), U1.5
- new net: Q4.2 (B), U2.5
- new net I_DISCHARGE: D2.1 (K), D3.1 (K), Q4.1 (C)
- new net THRESH: R5.1, R7.2, U3.1 (+)
Other:
- note added: ".model BC337 NPN(IS=4.13E-14 NF=0.9822 ISE=3.534E-15 NE=1.35 BF=292.4 IKF=0.9 VAF=145.7 NR=0.982 ISC=1.957E-13 NC=1.3 BR=23.68 IKR=0.1 VAR=20 RB=60 IRB=2.00E-04 RBM=8 RE=0.1129 RC=0.25 XTB=0 EG=1.11 XTI=3 CJE=3.799E-11 VJE=0.6752 MJE=0.3488 TF=5.4E-10 XTF=4 VTF=4.448 ITF=0.665 PTF=90 CJC=1.355E-11 VJC=0.3523 MJC=0.3831 XCJC=0.455 TR=3.00E-08 CJS=0 VJS=0.75 MJS=0.333 FC=0.643 Vceo=45 Icrating=500m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"
- note added: "Charing Current Source"
- note added: "Comparator Hysteresis"
- note added: "Control Voltage"
- note added: "Discharging Current Source"
- note added: "LM393"
- note added: "Oscillation Capacitor"
- note added: "Rectifier Switch"
- note added: "TS358 A"
- note added: "TS358 B"
- note removed: "BC327"
- note removed: "BC337"
