File: hardwired/oscilator/simple_transistor_saw/simple_transistor_saw/simple_transistor_saw.kicad_sch (KiCad schematic)
At the start: 0 parts

Commit message: Kicad version of simple transitor saw circuit
Parts:
- added C1: 0.01u, symbol Device:C
- added Q1, Q2: NPN, symbol Simulation_SPICE:NPN
- added R1, R2: 10k, symbol Device:R
- added R3: 50, symbol Device:R
- added R4: Potentiometer, symbol Simulation_SPICE:Potentiometer
- added R5: 22k, symbol Device:R
- added R6: 220, symbol Device:R
- added R7: 4.7k, symbol Device:R
- added U1, U2: ${SIM.PARAMS}, symbol Simulation_SPICE:OPAMP
- added V1, V2: 12, symbol Simulation_SPICE:VDC
Connections:
- new net: Q2.1 (C), R6.1
- new net: R1.1, R2.1, U2.1 (+)
- new net: R1.2, R5.1, R7.2, U2.5
- new net: Q1.2 (B), U1.5
- new net: Q1.3 (E), R3.1, U1.2 (-)
- new net: Q2.2 (B), R7.1
- new net +12V: R4.3, R5.2, R6.2, U1.3 (V+), U2.3 (V+), V1.1
- new net -12V: R3.2, U1.4 (V-), U2.4 (V-), V2.2
- new net 0: C1.2, R2.2, R4.1, V1.2, V2.1
- new net v_ramp: C1.1, Q1.1 (C), Q2.3 (E), U2.2 (-)
- new net vin_ctrl: R4.2, U1.1 (+)
