File: hardwired/oscilator/mosfet_saw/mosfet_saw.kicad_sch (KiCad schematic)
At the start: 23 parts, among them Q1 NPN, Q2 PNP, Q3 PNP, Q4 NPN, U1 ${SIM.PARAMS}, U2 ${SIM.PARAMS}, U3 ${SIM.PARAMS}, U4 ${SIM.PARAMS}

Commit message: Add improved breadboard PCB
Parts:
- removed Q1: NPN, symbol Simulation_SPICE:NPN
- added Q1: 2N7000, Package_TO_SOT_THT:TO-92_Inline, symbol Transistor_FET:2N7000
- R4: value 180k -> 100k
Connections:
- net D: now also Q1.3 (D)
- net GATE: now also Q1.2 (G)
- net S: now also Q1.1 (S)
